File: pcb/lqfp_adapters.sch (EAGLE design)
At the start: 21 parts, among them IC1 STM32F405RGT, IC2 STM32F303CBT, IC3 STM32F051K4T

Commit message: Added version 2 of the boards
Parts:
- removed SV1, SV3: (no value), con-lstb:MA20-1
- removed SV10, SV11, SV12, SV9: (no value), con-lstb:MA08-1
- removed SV13: (no value), con-lstb:MA05-2
- removed SV14, SV15: (no value), con-lstb:MA05-1
- removed SV16: (no value), con-lstb:MA10-2
- removed SV17, SV18: (no value), con-lstb:MA10-1
- removed SV2, SV4, SV5, SV6, SV7, SV8: (no value), con-lstb:MA12-1
- added SV-A1, SV-A4, SV-B1, SV-B2, SV-B3, SV-B4: (no value), MyComponents:MA12-1NO-PL
- added SV-A2, SV-A3: (no value), MyComponents:MA20-1NO-PL
- added SV-C1, SV-C3: (no value), MyComponents:MA05-1NO-PL
- added SV-C2: (no value), MyComponents:MA05-2
- added SV-D1, SVD3: (no value), MyComponents:MA10-1NO-PL
- added SV-D2: (no value), MyComponents:MA10-2
- added SV-E1, SV-E2, SV-E3, SV-E4: (no value), MyComponents:MA08-1NO-PL
- renumbered IC1 to IC-A1, IC2 to IC-B1, IC3 to IC-E1
Connections:
- net A1: now also SV-A2.1; no longer SV1.1
- net A10: now also SV-A2.10; no longer SV1.10
- net A11: now also SV-A2.11; no longer SV1.11
- net A12: now also SV-A2.12; no longer SV1.12
- net A13: now also SV-A2.13; no longer SV1.13
- net A14: now also SV-A2.14; no longer SV1.14
- net A15: now also SV-A2.15; no longer SV1.15
- net A16: now also SV-A2.16; no longer SV1.16
- net A17: now also SV-A2.17; no longer SV1.17
- net A18: now also SV-A2.18; no longer SV1.18
- net A19: now also SV-A2.19; no longer SV1.19
- net A2: now also SV-A2.2; no longer SV1.2
- net A20: now also SV-A2.20; no longer SV1.20
- net A21: now also SV-A1.1; no longer SV2.1
- net A22: now also SV-A1.2; no longer SV2.2
- net A23: now also SV-A1.3; no longer SV2.3
- net A24: now also SV-A1.4; no longer SV2.4
- net A25: now also SV-A1.5; no longer SV2.5
- net A26: now also SV-A1.6; no longer SV2.6
- net A27: now also SV-A1.7; no longer SV2.7
- net A28: now also SV-A1.8; no longer SV2.8
- net A29: now also SV-A1.9; no longer SV2.9
- net A3: now also SV-A2.3; no longer SV1.3
- net A30: now also SV-A1.10; no longer SV2.10
- net A31: now also SV-A1.11; no longer SV2.11
- net A32: now also SV-A1.12; no longer SV2.12
- net A33: now also SV-A3.1; no longer SV3.1
- net A34: now also SV-A3.2; no longer SV3.2
- net A35: now also SV-A3.3; no longer SV3.3
- net A36: now also SV-A3.4; no longer SV3.4
- net A37: now also SV-A3.5; no longer SV3.5
- net A38: now also SV-A3.6; no longer SV3.6
- net A39: now also SV-A3.7; no longer SV3.7
- net A4: now also SV-A2.4; no longer SV1.4
- net A40: now also SV-A3.8; no longer SV3.8
- net A41: now also SV-A3.9; no longer SV3.9
- net A42: now also SV-A3.10; no longer SV3.10
- net A43: now also SV-A3.11; no longer SV3.11
- net A44: now also SV-A3.12; no longer SV3.12
- net A45: now also SV-A3.13; no longer SV3.13
- net A46: now also SV-A3.14; no longer SV3.14
- net A47: now also SV-A3.15; no longer SV3.15
- net A48: now also SV-A3.16; no longer SV3.16
- net A49: now also SV-A3.17; no longer SV3.17
- net A5: now also SV-A2.5; no longer SV1.5
- net A50: now also SV-A3.18; no longer SV3.18
- net A51: now also SV-A3.19; no longer SV3.19
- net A52: now also SV-A3.20; no longer SV3.20
- net A53: now also SV-A4.1; no longer SV4.1
- net A54: now also SV-A4.2; no longer SV4.2
- net A55: now also SV-A4.3; no longer SV4.3
- net A56: now also SV-A4.4; no longer SV4.4
- net A57: now also SV-A4.5; no longer SV4.5
- net A58: now also SV-A4.6; no longer SV4.6
- net A59: now also SV-A4.7; no longer SV4.7
- net A6: now also SV-A2.6; no longer SV1.6
- net A60: now also SV-A4.8; no longer SV4.8
- net A61: now also SV-A4.9; no longer SV4.9
- net A62: now also SV-A4.10; no longer SV4.10
- net A63: now also SV-A4.11; no longer SV4.11
- net A64: now also SV-A4.12; no longer SV4.12
- net A7: now also SV-A2.7; no longer SV1.7
- net A8: now also SV-A2.8; no longer SV1.8
- net A9: now also SV-A2.9; no longer SV1.9
- net B1: now also SV-B2.1; no longer SV5.1
- net B10: now also SV-B2.10; no longer SV5.10
- net B11: now also SV-B2.11; no longer SV5.11
- net B12: now also SV-B2.12; no longer SV5.12
- net B13: now also SV-B1.1; no longer SV6.1
- net B14: now also SV-B1.2; no longer SV6.2
- net B15: now also SV-B1.3; no longer SV6.3
- net B16: now also SV-B1.4; no longer SV6.4
- net B17: now also SV-B1.5; no longer SV6.5
- net B18: now also SV-B1.6; no longer SV6.6
- net B19: now also SV-B1.7; no longer SV6.7
- net B2: now also SV-B2.2; no longer SV5.2
- net B20: now also SV-B1.8; no longer SV6.8
- net B21: now also SV-B1.9; no longer SV6.9
- net B22: now also SV-B1.10; no longer SV6.10
- net B23: now also SV-B1.11; no longer SV6.11
- net B24: now also SV-B1.12; no longer SV6.12
- net B25: now also SV-B3.1; no longer SV7.1
- net B26: now also SV-B3.2; no longer SV7.2
- net B27: now also SV-B3.3; no longer SV7.3
- net B28: now also SV-B3.4; no longer SV7.4
- net B29: now also SV-B3.5; no longer SV7.5
- net B3: now also SV-B2.3; no longer SV5.3
- net B30: now also SV-B3.6; no longer SV7.6
- net B31: now also SV-B3.7; no longer SV7.7
- net B32: now also SV-B3.8; no longer SV7.8
- net B33: now also SV-B3.9; no longer SV7.9
- net B34: now also SV-B3.10; no longer SV7.10
- net B35: now also SV-B3.11; no longer SV7.11
- net B36: now also SV-B3.12; no longer SV7.12
- net B37: now also SV-B4.1; no longer SV8.1
- net B38: now also SV-B4.2; no longer SV8.2
- net B39: now also SV-B4.3; no longer SV8.3
- net B4: now also SV-B2.4; no longer SV5.4
- net B40: now also SV-B4.4; no longer SV8.4
- net B41: now also SV-B4.5; no longer SV8.5
- net B42: now also SV-B4.6; no longer SV8.6
- net B43: now also SV-B4.7; no longer SV8.7
- net B44: now also SV-B4.8; no longer SV8.8
- net B45: now also SV-B4.9; no longer SV8.9
- net B46: now also SV-B4.10; no longer SV8.10
- net B47: now also SV-B4.11; no longer SV8.11
- net B48: now also SV-B4.12; no longer SV8.12
- net B5: now also SV-B2.5; no longer SV5.5
- net B6: now also SV-B2.6; no longer SV5.6
- net B7: now also SV-B2.7; no longer SV5.7
- net B8: now also SV-B2.8; no longer SV5.8
- net B9: now also SV-B2.9; no longer SV5.9
- net E1: now also SV-E2.1; no longer SV9.1
- net E10: now also SV-E1.2; no longer SV10.2
- net E11: now also SV-E1.3; no longer SV10.3
- net E12: now also SV-E1.4; no longer SV10.4
- net E13: now also SV-E1.5; no longer SV10.5
- net E14: now also SV-E1.6; no longer SV10.6
- net E15: now also SV-E1.7; no longer SV10.7
- net E16: now also SV-E1.8; no longer SV10.8
- net E17: now also SV-E3.1; no longer SV11.1
- net E18: now also SV-E3.2; no longer SV11.2
- net E19: now also SV-E3.3; no longer SV11.3
- net E2: now also SV-E2.2; no longer SV9.2
- net E20: now also SV-E3.4; no longer SV11.4
- net E21: now also SV-E3.5; no longer SV11.5
- net E22: now also SV-E3.6; no longer SV11.6
- net E23: now also SV-E3.7; no longer SV11.7
- net E24: now also SV-E3.8; no longer SV11.8
- net E25: now also SV-E4.1; no longer SV12.1
- net E26: now also SV-E4.2; no longer SV12.2
- net E27: now also SV-E4.3; no longer SV12.3
- net E28: now also SV-E4.4; no longer SV12.4
- net E29: now also SV-E4.5; no longer SV12.5
- net E3: now also SV-E2.3; no longer SV9.3
- net E30: now also SV-E4.6; no longer SV12.6
- net E31: now also SV-E4.7; no longer SV12.7
- net E32: now also SV-E4.8; no longer SV12.8
- net E4: now also SV-E2.4; no longer SV9.4
- net E5: now also SV-E2.5; no longer SV9.5
- net E6: now also SV-E2.6; no longer SV9.6
- net E7: now also SV-E2.7; no longer SV9.7
- net E8: now also SV-E2.8; no longer SV9.8
- net E9: now also SV-E1.1; no longer SV10.1
- net N$1: now also SV-C2.1, SV-C3.1; no longer SV13.1, SV15.1
- net N$10: now also SV-C1.5, SV-C2.10; no longer SV13.10, SV14.5
- net N$11: now also SV-D2.1, SVD3.1; no longer SV16.1, SV18.1
- net N$13: now also SV-D2.3, SVD3.2; no longer SV16.3, SV18.2
- net N$14: now also SV-D2.5, SVD3.3; no longer SV16.5, SV18.3
- net N$17: now also SV-D2.7, SVD3.4; no longer SV16.7, SV18.4
- net N$2: now also SV-C2.3, SV-C3.2; no longer SV13.3, SV15.2
- net N$22: now also SV-D2.9, SVD3.5; no longer SV16.9, SV18.5
- net N$23: now also SV-D2.11, SVD3.6; no longer SV16.11, SV18.6
- net N$24: now also SV-D2.13, SVD3.7; no longer SV16.13, SV18.7
- net N$25: now also SV-D2.15, SVD3.8; no longer SV16.15, SV18.8
- net N$26: now also SV-D2.17, SVD3.9; no longer SV16.17, SV18.9
- net N$27: now also SV-D2.19, SVD3.10; no longer SV16.19, SV18.10
- net N$28: now also SV-D1.10, SV-D2.20; no longer SV16.20, SV17.10
- net N$29: now also SV-D1.9, SV-D2.18; no longer SV16.18, SV17.9
- net N$3: now also SV-C2.5, SV-C3.3; no longer SV13.5, SV15.3
- net N$31: now also SV-D1.8, SV-D2.16; no longer SV16.16, SV17.8
- net N$32: now also SV-D1.7, SV-D2.14; no longer SV16.14, SV17.7
- net N$33: now also SV-D1.6, SV-D2.12; no longer SV16.12, SV17.6
- net N$34: now also SV-D1.5, SV-D2.10; no longer SV16.10, SV17.5
- net N$35: now also SV-D1.4, SV-D2.8; no longer SV16.8, SV17.4
- net N$36: now also SV-D1.3, SV-D2.6; no longer SV16.6, SV17.3
- net N$37: now also SV-D1.2, SV-D2.4; no longer SV16.4, SV17.2
- net N$38: now also SV-D1.1, SV-D2.2; no longer SV16.2, SV17.1
- net N$4: now also SV-C2.7, SV-C3.4; no longer SV13.7, SV15.4
- net N$5: now also SV-C2.9, SV-C3.5; no longer SV13.9, SV15.5
- net N$6: now also SV-C1.1, SV-C2.2; no longer SV13.2, SV14.1
- net N$7: now also SV-C1.2, SV-C2.4; no longer SV13.4, SV14.2
- net N$8: now also SV-C1.3, SV-C2.6; no longer SV13.6, SV14.3
- net N$9: now also SV-C1.4, SV-C2.8; no longer SV13.8, SV14.4
