File: pcb/stm32_pi_board.sch (EAGLE design)
At the start: 63 parts, among them IC1 LD1117, IC2 ESP-11, IC3 LD1117, IC4 STM32F405RG, IC5 STF203-22, Q1 BSH205, Q2 N2004, Q5 BSH205, X1 PJ-043-SMT, X2 DM3AT, X3 XM7D-0512

Commit message: Updated PCB
Parts:
- removed SV5: 69190-410HLF, MyComponents:MA10-1NO-PL
- added SV3: (no value), MyComponents:MA12-1NO-PL
Connections:
- net GND: now also SV3.2; no longer SV5.1
- net PA0: now also SV3.3; no longer SV5.2
- net PB4: now also SV3.11; no longer SV5.10
- net PB5: now also SV3.10; no longer SV5.9
- net PB6: now also SV3.9; no longer SV5.8
- net PB7: now also SV3.8; no longer SV5.7
- net PB8: now also SV3.7; no longer SV5.6
- net PB9: now also SV3.6; no longer SV5.5
- net PC0: now also SV3.4; no longer SV5.3
- net PC13: now also SV3.5; no longer SV5.4
- net USB-VBUS: now also SV3.12
- net VIN: now also SV3.1
Changed lines of the file:
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@@
 <setting verticaltext="up"/>
 </settings>
-<grid distance="0.1" unitdist="inch" unit="inch" style="lines" multiple="1" display="no" altdistance="0.01" altunitdist="inch" altunit="inch"/>
+<grid distance="0.1" unitdist="inch" unit="inch" style="lines" multiple="1" display="yes" altdistance="0.01" altunitdist="inch" altunit="inch"/>
 <layers>
 <layer number="1" name="Top" color="4" fill="1" visible="no" active="no"/>
@@
 <part name="C12" library="MyComponents" deviceset="C-US" device="0805" value="0.1uF"/>
 <part name="SV4" library="MyComponents" deviceset="MA20-1" device="NO-PL" value="68000-420HLF"/>
-<part name="SV5" library="MyComponents" deviceset="MA10-1" device="NO-PL" value="69190-410HLF"/>
 <part name="D1" library="MyComponents" deviceset="RGB-LED-5MM" device="" value="WP154A4SUREQBFZGC"/>
 <part name="R6" library="MyComponents" deviceset="R-US" device="0805" value="330"/>
@@
 <part name="SUPPLY42" library="supply2" deviceset="VCC" device=""/>
 <part name="SUPPLY43" library="supply2" deviceset="GND" device=""/>
+<part name="SV3" library="MyComponents" deviceset="MA12-1" device="NO-PL"/>
 </parts>
 <sheets>
@@
 <instance part="C12" gate="G$1" x="261.62" y="147.32" rot="R180"/>
 <instance part="SV4" gate="1" x="198.12" y="78.74" rot="R180"/>
-<instance part="SV5" gate="1" x="246.38" y="78.74" rot="R180"/>
 <instance part="D1" gate="1" x="43.18" y="154.94" smashed="yes">
 <attribute name="NAME" x="48.26" y="144.78" size="1.27" layer="95" rot="R180"/>
@@
 <instance part="SUPPLY42" gate="G$1" x="185.42" y="50.8" rot="R180"/>
 <instance part="SUPPLY43" gate="GND" x="218.44" y="86.36"/>
+<instance part="SV3" gate="1" x="246.38" y="78.74" rot="R180"/>
 </instances>
 <busses>
@@
 </segment>
 <segment>
-<pinref part="SV5" gate="1" pin="1"/>
 <pinref part="SUPPLY43" gate="GND" pin="GND"/>
 <wire x1="238.76" y1="88.9" x2="218.44" y2="88.9" width="0.1524" layer="91"/>
+<pinref part="SV3" gate="1" pin="2"/>
 </segment>
 </net>
@@
 <junction x="147.32" y="254"/>
 <label x="132.08" y="254" size="1.27" layer="95"/>
+</segment>
+<segment>
+<pinref part="SV3" gate="1" pin="1"/>
+<wire x1="238.76" y1="91.44" x2="226.06" y2="91.44" width="0.1524" layer="91"/>
+<label x="233.68" y="91.44" size="1.27" layer="95" rot="R180"/>
 </segment>
 </net>
@@
 <wire x1="238.76" y1="83.82" x2="226.06" y2="83.82" width="0.1524" layer="91"/>
 <label x="233.68" y="83.82" size="1.27" layer="95" rot="R180"/>
-<pinref part="SV5" gate="1" pin="3"/>
+<pinref part="SV3" gate="1" pin="4"/>
 </segment>
 </net>
@@
 <label x="137.16" y="129.54" size="1.27" layer="95"/>
 </segment>
+<segment>
+<pinref part="SV3" gate="1" pin="12"/>
+<wire x1="238.76" y1="63.5" x2="226.06" y2="63.5" width="0.1524" layer="91"/>
+<label x="233.68" y="63.5" size="1.27" layer="95" rot="R180"/>
+</segment>
 </net>
 <net name="USB-DM" class="0">
@@
 </segment>
 <segment>
-<pinref part="SV5" gate="1" pin="10"/>
 <wire x1="238.76" y1="66.04" x2="226.06" y2="66.04" width="0.1524" layer="91"/>
 <label x="233.68" y="66.04" size="1.27" layer="95" rot="R180"/>
+<pinref part="SV3" gate="1" pin="11"/>
 </segment>
 </net>
@@
 </segment>
 <segment>
-<pinref part="SV5" gate="1" pin="9"/>
 <wire x1="238.76" y1="68.58" x2="226.06" y2="68.58" width="0.1524" layer="91"/>
 <label x="233.68" y="68.58" size="1.27" layer="95" rot="R180"/>
+<pinref part="SV3" gate="1" pin="10"/>
 </segment>
 </net>
@@
 </segment>
 <segment>
-<pinref part="SV5" gate="1" pin="8"/>
 <wire x1="238.76" y1="71.12" x2="226.06" y2="71.12" width="0.1524" layer="91"/>
 <label x="233.68" y="71.12" size="1.27" layer="95" rot="R180"/>
+<pinref part="SV3" gate="1" pin="9"/>
 </segment>
 </net>
@@
 </segment>
 <segment>
-<pinref part="SV5" gate="1" pin="7"/>
 <wire x1="238.76" y1="73.66" x2="226.06" y2="73.66" width="0.1524" layer="91"/>
 <label x="233.68" y="73.66" size="1.27" layer="95" rot="R180"/>
+<pinref part="SV3" gate="1" pin="8"/>
 </segment>
 </net>
@@
 </segment>
 <segment>
-<pinref part="SV5" gate="1" pin="6"/>
 <wire x1="238.76" y1="76.2" x2="226.06" y2="76.2" width="0.1524" layer="91"/>
 <label x="233.68" y="76.2" size="1.27" layer="95" rot="R180"/>
+<pinref part="SV3" gate="1" pin="7"/>
 </segment>
 </net>
@@
 </segment>
 <segment>
-<pinref part="SV5" gate="1" pin="5"/>
 <wire x1="238.76" y1="78.74" x2="226.06" y2="78.74" width="0.1524" layer="91"/>
 <label x="233.68" y="78.74" size="1.27" layer="95" rot="R180"/>
+<pinref part="SV3" gate="1" pin="6"/>
 </segment>
 </net>
@@
 <wire x1="238.76" y1="81.28" x2="226.06" y2="81.28" width="0.1524" layer="91"/>
 <label x="233.68" y="81.28" size="1.27" layer="95" rot="R180"/>
-<pinref part="SV5" gate="1" pin="4"/>
+<pinref part="SV3" gate="1" pin="5"/>
 </segment>
 <segment>
@@
 <wire x1="238.76" y1="86.36" x2="226.06" y2="86.36" width="0.1524" layer="91"/>
 <label x="233.68" y="86.36" size="1.27" layer="95" rot="R180"/>
-<pinref part="SV5" gate="1" pin="2"/>
-</segment>
-</net>
+<pinref part="SV3" gate="1" pin="3"/>
+</segment>
+</net>

Commit message: Revision 1.1 submitted to factory
Parts:
- removed ESP-PWR: (no value), MyComponents:MA03-1PL
- removed IC1: LD1117, MyComponents:REG1117
- removed Q1: BSH205, MyComponents:BSH205G2R
- removed Q2: N2004, MyComponents:N2004
- removed R1: 1.4M, MyComponents:R-US0805
- removed R2: 330K, MyComponents:R-US0805
- added IC6: MIC5219-3.3, v-reg-micrel:MIC5219XX
- added PWR: (no value), MyComponents:MA03-1PL
- C2: value 0.1uF -> 470pF
- C3: value 10uF -> 2.2uF
- renumbered LED1 to ESP-ON, LED2 to SD-ON
Connections:
- removed net E_VG: Q1.G, Q2.D, R1.1
- removed net N$148: C2.2, IC1.VIN, Q1.D
- removed net N$150: Q2.S, R3.2
- new net N$4: C2.2, IC6.BYP
- net ESP-ON: now also PWR.3; no longer ESP-PWR.3
- net ESP-ON1: now also IC6.EN, PWR.2, R3.2; no longer ESP-PWR.2, Q2.G, R2.2
- net ESP-VDD: now also IC6.OUT; no longer IC1.VOUT
- net GND: now also IC6.GND; no longer IC1.GND, R2.1
- net VDD: now also PWR.1; no longer ESP-PWR.1
- net VIN: now also IC6.IN; no longer Q1.S, R1.2
Other:
- note removed: "Vmax = min(V(N2004) + V(LD1117)) = 20V+15V = 15V"
- moved on the sheet: C2, C3, R3

Commit message: Assembled board 1.2
Parts:
- added C20, C21, C25, C26, C28, C29, C30, C31, C33: 0.1uF, MyComponents:C-US0805
- added C22: 2.2uF, MyComponents:CPOL-US0805
- added C23: 470pF, MyComponents:C-US0805
- added C24, C27, C35, C36, C37: 47uF, MyComponents:CPOL-US1311
- added C32, C34: 1.0uF, MyComponents:C-US0805
- added IC1, IC8: MIC5219-3.3, MyComponents:MIC5219XX
- added IC7: IS31AP2005, MyComponents:IS31AP2005
- added IC9: UDA1334ATS, MyComponents:UDA1334ATS
- added Q1: FDG6332C, MyComponents:N-P-MOS
- added R1, R2, R20, R21, R9: 150K, MyComponents:R-US0805
- added R11: 6.7K, MyComponents:R-US0805
- added R12, R18: 1, MyComponents:R-US0805
- added R19, R24, R25: 10K, MyComponents:R-US0805
- added R22, R23: 220K, MyComponents:R-US0805
- added SV5: (no value), MyComponents:MA04-1PL
- C3: device MyComponents:C-US0805 -> MyComponents:CPOL-US0805
- C6: value 0.1uF -> 470pF
- C7: value 10uF -> 2.2uF; device MyComponents:C-US0805 -> MyComponents:CPOL-US0805
- HSE: device MyComponents:Q-HC-46X -> MyComponents:Q-HSEFA-128
- IC3: value LD1117 -> IS31AP2005; device MyComponents:REG1117 -> MyComponents:IS31AP2005
- IC6: device v-reg-micrel:MIC5219XX -> MyComponents:MIC5219XX
- LSE: device MyComponents:Q-MC-306 -> MyComponents:Q-LSECM7V-T1A
- R7: value 150 -> 100
Connections:
- removed net PB10: IC4MCU.PB10, SV4.10
- removed net PB11: IC4MCU.PB11, SV4.9
- removed net PB12: IC4MCU.PB12, SV4.8
- removed net PB13: IC4MCU.PB13, SV4.7
- removed net PB14: IC4MCU.PB14, SV4.6
- removed net PB15: IC4MCU.PB15, SV4.5
- new net AUD-BCK: IC4MCU.PB10, IC9.BCK, SV4.10
- new net AUD-DAT: IC4MCU.PB15, IC9.DATAI, SV4.5
- new net AUD-L: C35.+, IC9.VOUTL
- new net AUD-MUTE: IC4MCU.PB13, IC9.MUTE, R19.1, SV4.7
- new net AUD-ON: IC4MCU.PB11, IC8.EN, Q1.2, R24.1, SV4.9
- new net AUD-R: C36.+, IC9.VOUTR
- new net AUD-REF: C24.+, C25.1, IC9.VREFDAC, R11.1, R9.2
- new net AUD-SMPL: IC4MCU.PB14, IC9.SYSCLK, SV4.6
- new net AUD-WS: IC4MCU.PB12, IC9.WS, SV4.8
- new net N$11: IC3.OUT-, SV5.1
- new net N$13: IC3.OUT+, SV5.2
- new net N$17: C20.1, R1.2
- new net N$22: IC7.OUT-, SV5.3
- new net N$24: IC7.OUT+, SV5.4
- new net N$26: IC3.IN+, R1.1
- new net N$27: IC7.IN+, R2.1
- new net N$37: C21.1, R2.2
- new net N$38: IC3.IN-, R20.1
- new net N$42: C28.1, C37.+, IC9.VCC, R18.1
- new net N$43: IC7.IN-, R21.1
- new net N$44: C23.2, IC8.BYP
- new net N$46: C26.1, C27.+, IC9.VSS, R12.1
- new net N$47: C30.1, R21.2
- new net N$5: C6.2, IC1.BYP
- new net N$65: C29.1, R20.2
- new net N$69: C29.2, C35.-, R22.2
- new net N$70: Q1.3, R18.2
- new net N$72: C30.2, C36.-, R23.2
- new net N$86: Q1.5, Q1.6, R25.2
- new net VSS: C22.+, C31.1, C32.1, C33.1, C34.1, IC3.SDB, IC3.VSS, IC7.SDB, IC7.VSS, IC8.OUT, R12.2, R9.1
- net ESP-VDD: now also C3.+; no longer C3.2
- net GND: now also C20.2, C21.2, C22.-, C23.1, C24.-, C25.2, C26.2, C27.-, C28.2, C3.-, C31.2, C32.2, C33.2, C34.2, C37.-, C7.-, IC1.GND, IC3.AGND, IC7.AGND, IC8.GND, IC9.AGND, IC9.DEEM, IC9.GND, IC9.PLL0, IC9.SFOR0, IC9.SFOR1, Q1.1, R11.2, R19.2, R22.1, R23.1, R24.2; no longer C3.1, C7.1, IC3.GND
- net VDD: now also C7.+, IC1.OUT, Q1.4, R25.1; no longer C7.2, IC3.VOUT, PWR.1
- net VIN: now also IC1.EN, IC1.IN, IC8.IN, PWR.1; no longer C6.2, IC3.VIN
