File: pcb/stm32_pi_board.sch (EAGLE design)
At the start: 102 parts, among them IC1 LMT86, IC10 REG1117, IC2 ESP-11, IC3 IS31AP2005, IC4 STM32F405RG, IC5 STF203-22, IC6 MIC5219-3.3, IC7 IS31AP2005, IC8 MIC5219-3.3, IC9 UDA1334ATS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

Commit message: PCB revision 1.3
Parts:
- added C40: 470 uF, MyComponents:CPOL-US2917
Connections:
- net GND: now also C40.-
- net VIN: now also C40.+
Changed lines of the file:
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@@
 <setting verticaltext="up"/>
 </settings>
-<grid distance="0.1" unitdist="inch" unit="inch" style="lines" multiple="1" display="no" altdistance="0.01" altunitdist="inch" altunit="inch"/>
+<grid distance="0.1" unitdist="inch" unit="inch" style="lines" multiple="1" display="yes" altdistance="0.01" altunitdist="inch" altunit="inch"/>
 <layers>
 <layer number="1" name="Top" color="4" fill="1" visible="no" active="no"/>
@@
 <part name="C39" library="rcl" deviceset="C-EU" device="C1206" value="0.1 uF"/>
 <part name="SUPPLY20" library="supply2" deviceset="VCC" device=""/>
+<part name="C40" library="MyComponents" deviceset="CPOL-US" device="2917" value="470 uF"/>
 </parts>
 <sheets>
@@
 </instance>
 <instance part="C38" gate="G$1" x="177.8" y="149.86" smashed="yes" rot="R90">
-<attribute name="NAME" x="177.165" y="150.495" size="1.27" layer="95" rot="R180" align="top-left"/>
-<attribute name="VALUE" x="180.34" y="149.225" size="1.27" layer="96" align="top-left"/>
+<attribute name="NAME" x="177" y="150.5" size="1.27" layer="95" rot="R180" align="top-left"/>
+<attribute name="VALUE" x="180" y="149.5" size="1.27" layer="96" align="top-left"/>
 </instance>
 <instance part="D1" gate="1" x="340.36" y="236.22" rot="R180"/>
@@
 <instance part="SUPPLY20" gate="G$1" x="401.32" y="177.8" smashed="yes" rot="R180">
 <attribute name="VALUE" x="403.225" y="174.625" size="1.27" layer="96" rot="R180"/>
+</instance>
+<instance part="C40" gate="G$1" x="177.8" y="137.16" smashed="yes" rot="R90">
+<attribute name="NAME" x="177" y="138" size="1.27" layer="95" align="bottom-right"/>
+<attribute name="VALUE" x="180" y="136.5" size="1.27" layer="96" rot="R180" align="bottom-right"/>
 </instance>
 </instances>
@@
 <wire x1="187.96" y1="154.94" x2="187.96" y2="149.86" width="0.1524" layer="91"/>
 <junction x="187.96" y="127"/>
-<wire x1="187.96" y1="149.86" x2="187.96" y2="127" width="0.1524" layer="91"/>
+<wire x1="187.96" y1="149.86" x2="187.96" y2="137.16" width="0.1524" layer="91"/>
 <pinref part="C7" gate="G$1" pin="-"/>
+<wire x1="187.96" y1="137.16" x2="187.96" y2="127" width="0.1524" layer="91"/>
 <wire x1="228.6" y1="142.24" x2="228.6" y2="137.16" width="0.1524" layer="91"/>
 <pinref part="C38" gate="G$1" pin="2"/>
@@
 <wire x1="218.44" y1="137.16" x2="228.6" y2="137.16" width="0.1524" layer="91"/>
 <junction x="228.6" y="137.16"/>
+<pinref part="C40" gate="G$1" pin="-"/>
+<wire x1="182.88" y1="137.16" x2="187.96" y2="137.16" width="0.1524" layer="91"/>
+<junction x="187.96" y="137.16"/>
 </segment>
 <segment>
@@
 <wire x1="172.72" y1="149.86" x2="175.26" y2="149.86" width="0.1524" layer="91"/>
 <label x="170.18" y="170.18" size="1.27" layer="95"/>
+<pinref part="C40" gate="G$1" pin="+"/>
+<wire x1="175.26" y1="137.16" x2="172.72" y2="137.16" width="0.1524" layer="91"/>
+<wire x1="172.72" y1="137.16" x2="172.72" y2="149.86" width="0.1524" layer="91"/>
+<junction x="172.72" y="149.86"/>
 </segment>
 </net>

Commit message: Revision 1.3 of Stm32-Pi-Board
Parts:
- added OPH1: AMS3, photo-elements:VT935GB
- added R29: 4.7K, MyComponents:R-US0805
- C39: device rcl:C-EUC1206 -> MyComponents:C-US0805
Connections:
- net GND: now also R29.1
- net PC0: now also OPH1.1, R29.2
- net VDD: now also OPH1.2
Changed lines of the file:
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@@
 <setting verticaltext="up"/>
 </settings>
-<grid distance="0.1" unitdist="inch" unit="inch" style="lines" multiple="1" display="yes" altdistance="0.01" altunitdist="inch" altunit="inch"/>
+<grid distance="0.1" unitdist="inch" unit="inch" style="lines" multiple="1" display="no" altdistance="0.01" altunitdist="inch" altunit="inch"/>
 <layers>
-<layer number="1" name="Top" color="4" fill="1" visible="no" active="no"/>
-<layer number="16" name="Bottom" color="1" fill="1" visible="no" active="no"/>
-<layer number="17" name="Pads" color="2" fill="1" visible="no" active="no"/>
-<layer number="18" name="Vias" color="2" fill="1" visible="no" active="no"/>
-<layer number="19" name="Unrouted" color="6" fill="1" visible="no" active="no"/>
-<layer number="20" name="Dimension" color="15" fill="1" visible="no" active="no"/>
-<layer number="21" name="tPlace" color="7" fill="1" visible="no" active="no"/>
-<layer number="22" name="bPlace" color="7" fill="1" visible="no" active="no"/>
-<layer number="23" name="tOrigins" color="15" fill="1" visible="no" active="no"/>
-<layer number="24" name="bOrigins" color="15" fill="1" visible="no" active="no"/>
-<layer number="25" name="tNames" color="7" fill="1" visible="no" active="no"/>
-<layer number="26" name="bNames" color="7" fill="1" visible="no" active="no"/>
-<layer number="27" name="tValues" color="7" fill="1" visible="no" active="no"/>
-<layer number="28" name="bValues" color="7" fill="1" visible="no" active="no"/>
+<layer number="1" name="Top" color="4" fill="1" visible="yes" active="no"/>
+<layer number="16" name="Bottom" color="1" fill="1" visible="yes" active="no"/>
+<layer number="17" name="Pads" color="2" fill="1" visible="yes" active="no"/>
+<layer number="18" name="Vias" color="2" fill="1" visible="yes" active="no"/>
+<layer number="19" name="Unrouted" color="6" fill="1" visible="yes" active="no"/>
+<layer number="20" name="Dimension" color="15" fill="1" visible="yes" active="no"/>
+<layer number="21" name="tPlace" color="7" fill="1" visible="yes" active="no"/>
+<layer number="22" name="bPlace" color="7" fill="1" visible="yes" active="no"/>
+<layer number="23" name="tOrigins" color="15" fill="1" visible="yes" active="no"/>
+<layer number="24" name="bOrigins" color="15" fill="1" visible="yes" active="no"/>
+<layer number="25" name="tNames" color="7" fill="1" visible="yes" active="no"/>
+<layer number="26" name="bNames" color="7" fill="1" visible="yes" active="no"/>
+<layer number="27" name="tValues" color="7" fill="1" visible="yes" active="no"/>
+<layer number="28" name="bValues" color="7" fill="1" visible="yes" active="no"/>
 <layer number="29" name="tStop" color="7" fill="3" visible="no" active="no"/>
 <layer number="30" name="bStop" color="7" fill="6" visible="no" active="no"/>
@@
 <layer number="35" name="tGlue" color="7" fill="4" visible="no" active="no"/>
 <layer number="36" name="bGlue" color="7" fill="5" visible="no" active="no"/>
-<layer number="37" name="tTest" color="7" fill="1" visible="no" active="no"/>
-<layer number="38" name="bTest" color="7" fill="1" visible="no" active="no"/>
+<layer number="37" name="tTest" color="7" fill="1" visible="yes" active="no"/>
+<layer number="38" name="bTest" color="7" fill="1" visible="yes" active="no"/>
 <layer number="39" name="tKeepout" color="4" fill="11" visible="no" active="no"/>
 <layer number="40" name="bKeepout" color="1" fill="11" visible="no" active="no"/>
@@
 <layer number="44" name="Drills" color="7" fill="1" visible="no" active="no"/>
 <layer number="45" name="Holes" color="7" fill="1" visible="no" active="no"/>
-<layer number="46" name="Milling" color="3" fill="1" visible="no" active="no"/>
-<layer number="47" name="Measures" color="7" fill="1" visible="no" active="no"/>
-<layer number="48" name="Document" color="7" fill="1" visible="no" active="no"/>
-<layer number="49" name="Reference" color="7" fill="1" visible="no" active="no"/>
-<layer number="50" name="dxf" color="7" fill="1" visible="no" active="no"/>
-<layer number="51" name="tDocu" color="7" fill="1" visible="no" active="no"/>
-<layer number="52" name="bDocu" color="7" fill="1" visible="no" active="no"/>
-<layer number="53" name="tGND_GNDA" color="7" fill="9" visible="no" active="no"/>
-<layer number="54" name="bGND_GNDA" color="1" fill="9" visible="no" active="no"/>
-<layer number="56" name="wert" color="7" fill="1" visible="no" active="no"/>
+<layer number="46" name="Milling" color="3" fill="1" visible="yes" active="no"/>
+<layer number="47" name="Measures" color="7" fill="1" visible="yes" active="no"/>
+<layer number="48" name="Document" color="7" fill="1" visible="yes" active="no"/>
+<layer number="49" name="Reference" color="7" fill="1" visible="yes" active="no"/>
+<layer number="50" name="dxf" color="7" fill="1" visible="yes" active="no"/>
+<layer number="51" name="tDocu" color="7" fill="1" visible="yes" active="no"/>
+<layer number="52" name="bDocu" color="7" fill="1" visible="yes" active="no"/>
+<layer number="53" name="tGND_GNDA" color="7" fill="9" visible="yes" active="no"/>
+<layer number="54" name="bGND_GNDA" color="1" fill="9" visible="yes" active="no"/>
+<layer number="56" name="wert" color="7" fill="1" visible="yes" active="no"/>
 <layer number="90" name="Modules" color="5" fill="1" visible="yes" active="yes"/>
 <layer number="91" name="Nets" color="2" fill="1" visible="yes" active="yes"/>
@@
 <part name="IC1" library="MyComponents" deviceset="LMT86" device=""/>
 <part name="SUPPLY19" library="supply2" deviceset="GND" device=""/>
-<part name="C39" library="rcl" deviceset="C-EU" device="C1206" value="0.1 uF"/>
+<part name="C39" library="MyComponents" deviceset="C-US" device="0805" value="0.1 uF"/>
 <part name="SUPPLY20" library="supply2" deviceset="VCC" device=""/>
 <part name="C40" library="MyComponents" deviceset="CPOL-US" device="2917" value="470 uF"/>
+<part name="R29" library="MyComponents" deviceset="R-US" device="0805" value="4.7K"/>
+<part name="OPH1" library="photo-elements" deviceset="VT9" device="" technology="35GB" value="AMS3"/>
+<part name="SUPPLY21" library="supply2" deviceset="GND" device=""/>
+<part name="SUPPLY22" library="supply2" deviceset="VCC" device=""/>
 </parts>
 <sheets>
@@
 <attribute name="NAME" x="177" y="138" size="1.27" layer="95" align="bottom-right"/>
 <attribute name="VALUE" x="180" y="136.5" size="1.27" layer="96" rot="R180" align="bottom-right"/>
+</instance>
+<instance part="R29" gate="G$1" x="388.62" y="218.44" rot="R90"/>
+<instance part="OPH1" gate="G$1" x="388.62" y="233.68" rot="R180"/>
+<instance part="SUPPLY21" gate="GND" x="388.62" y="208.28"/>
+<instance part="SUPPLY22" gate="G$1" x="388.62" y="243.84" smashed="yes">
+<attribute name="VALUE" x="386.715" y="247.015" size="1.27" layer="96"/>
 </instance>
 </instances>
@@
 <junction x="401.32" y="195.58"/>
 </segment>
+<segment>
+<pinref part="SUPPLY21" gate="GND" pin="GND"/>
+<pinref part="R29" gate="G$1" pin="1"/>
+<wire x1="388.62" y1="210.82" x2="388.62" y2="213.36" width="0.1524" layer="91"/>
+</segment>
 </net>
 <net name="VIN" class="0">
@@
 <junction x="401.32" y="182.88"/>
 </segment>
+<segment>
+<pinref part="SUPPLY22" gate="G$1" pin="VCC"/>
+<pinref part="OPH1" gate="G$1" pin="2"/>
+<wire x1="388.62" y1="241.3" x2="388.62" y2="238.76" width="0.1524" layer="91"/>
+</segment>
 </net>
 <net name="NRST" class="0">
@@
 <label x="233.68" y="76.2" size="1.27" layer="95" rot="R180"/>
 </segment>
-</net>
+<segment>
+<pinref part="OPH1" gate="G$1" pin="1"/>
+<pinref part="R29" gate="G$1" pin="2"/>
+<wire x1="388.62" y1="228.6" x2="388.62" y2="226.06" width="0.1524" layer="91"/>
+<wire x1="388.62" y1="226.06" x2="388.62" y2="223.52" width="0.1524" layer="91"/>
+<wire x1="388.62" y1="226.06" x2="373.38" y2="226.06" width="0.1524" layer="91"/>
+<junction x="388.62" y="226.06"/>
+<label x="373.38" y="226.06" size="1.778" layer="95"/>
+</segment>
+</net>

Commit message: Submitted PiBoard v1.3
Connections:
- net GND: no longer D1.C
- net N$5: now also D1.AR; no longer D1.AG
- net N$75: now also D1.AG; no longer D1.AR
- net VDD: now also D1.C
Other:
- moved on the sheet: R27, R6
