File: pcb/stm_adapters.sch (EAGLE design)
At the start: 65 parts, among them IC1 STM32F405RGT, IC2 STM32F303CBT, IC3 STM32F303x6/x8, IC5 TL431, J1 BUTTON-FSM14JRT, J2 BUTTON-FSM14JRT, J3 BUTTON-FSM14JRT, Q11 32.7680kHz, Q21 32.7680kHz

Commit message: Added version 2 of the boards
Parts:
- removed IC5: TL431, MyComponents:TL431CL3T
- removed R14: 220, rcl:R-EU_R1206
- removed R2, R3: 0K, rcl:R-EU_R1206
- removed SV17, SV18: (no value), con-lstb:MA10-1
- added L1, L2, L3, L4, L5, L6: (no value), MyComponents:L-US0603
- added R10, R32: 10K, MyComponents:R-US0805
- added R20, R30: 0, MyComponents:R-US0805
- added RQ: 220, MyComponents:R-US0805
- added SV19: (no value), MyComponents:MA09-1NO-PL
- added SV5: (no value), MyComponents:MA07-1NO-PL
- C1: value 4.7uF -> P30; device rcl:C-EUC1206 -> MyComponents:C-US0805
- C11, C14, C15, C2, C22, C3, C32: device rcl:C-EUC1206 -> MyComponents:C-US0805
- C12, C13, C16, C19, C21, C23, C27, C28, C30, C31, C35: value 100nF -> 0.1uF; device rcl:C-EUC1206 -> MyComponents:C-US0805
- C24, C25, C33, C34: value 10pF -> 12pF; device rcl:C-EUC1206 -> MyComponents:C-US0805
- Q1, Q2, Q3: value (none) -> HSE; device MyComponents:HC-46X -> MyComponents:Q-HC-46X
- Q11, Q21: value 32.7680kHz -> LSE; device crystal:MC-306 -> MyComponents:Q-MC-306
- R11: value 0K -> 0; device rcl:R-EU_R1206 -> MyComponents:R-US0805
- R12: value 0K -> P31; device rcl:R-EU_R1206 -> MyComponents:R-US0805
- R13: value 0K -> P47; device rcl:R-EU_R1206 -> MyComponents:R-US0805
- R15, R22, R31, R40, R41, R42: device rcl:R-EU_R1206 -> MyComponents:R-US0805
- R21: value 330 -> 10K; device rcl:R-EU_R1206 -> MyComponents:R-US0805
- SV1, SV3: device con-lstb:MA20-1 -> MyComponents:MA20-1NO-PL
- SV10, SV11: device con-lstb:MA08-1 -> MyComponents:MA08-1NO-PL
- SV12: device con-lstb:MA08-1 -> MyComponents:MA09-1NO-PL
- SV13, SV14, SV15, SV4: device con-lstb:MA05-2 -> MyComponents:MA05-2
- SV16: device con-lstb:MA10-2 -> MyComponents:MA10-2
- SV2, SV8: device con-lstb:MA07-1 -> MyComponents:MA07-1NO-PL
- SV6, SV7: device con-lstb:MA12-1 -> MyComponents:MA12-1NO-PL
- SV9: device con-lstb:MA08-1 -> MyComponents:MA07-1NO-PL
Connections:
- net N$64 renamed ACAP1
- net N$65 renamed ACAP2
- new net N$10: L6.2, SV16.15
- new net N$11: L5.2, SV16.13
- new net N$13: L4.2, SV16.9
- new net N$24: L3.2, SV16.7
- new net N$29: L2.2, SV16.5
- new net N$36: L1.2, SV16.3
- net AD_RST: now also L6.1; no longer SV16.15
- net AD_TCK: now also L4.1; no longer SV16.9
- net AD_TDI: now also L2.1; no longer SV16.5
- net AD_TDO: now also L5.1; no longer SV16.13
- net AD_TMS: now also L3.1; no longer SV16.7
- net AD_TRST: now also L1.1; no longer SV16.3
- net ARST: now also R10.1
- net AVDD: now also R10.2
- net AVSS: now also SV4.5
- net B10: now also SV12.7; no longer SV17.8
- net B11: now also SV12.8; no longer SV17.9
- net B12: now also SV12.9; no longer SV17.10
- net B2: now also SV12.5; no longer SV17.6
- net B36: now also SV19.1; no longer SV18.1
- net B41: now also SV19.6; no longer SV18.6
- net B42: now also SV19.7; no longer SV18.7
- net B43: now also SV19.8; no longer SV18.8
- net B45: now also SV12.3; no longer SV17.4
- net B46: now also SV12.4; no longer SV17.5
- net BBAT: now also R20.1; no longer R2.1
- net BBOOT: now also R21.1, SV12.2; no longer R22.1, SV17.3
- net BRST: now also R22.2, SV12.6; no longer SV17.7
- net BTCK: now also SV19.2; no longer SV18.2
- net BTDI: now also SV19.3; no longer SV18.3
- net BTDO: now also SV19.4; no longer SV18.4
- net BTRST: now also SV19.5; no longer SV18.5
- net BVDD: now also R20.2, R22.1; no longer R2.2, R21.2
- net BVREF: no longer IC5.C, IC5.R, R21.1
- net BVSS: now also R21.2, SV12.1, SV19.9; no longer IC5.A, R22.2, SV17.1, SV18.10
- net E28: now also SV9.4; no longer SV12.4
- net E29: now also SV9.5; no longer SV12.5
- net E30: now also SV9.6; no longer SV12.6
- net E6: now also SV5.5; no longer SV9.6
- net E7: now also SV5.6; no longer SV9.7
- net E8: now also SV5.7; no longer SV9.8
- net EBOOT: now also SV5.2; no longer SV9.3
- net ERST: now also R32.2, SV5.3; no longer SV9.4
- net ETDI: now also SV9.1; no longer SV12.1
- net ETDO: now also SV9.2; no longer SV12.2
- net ETRST: now also SV9.3; no longer SV12.3
- net EVDD: now also R30.2, R32.1; no longer R3.2
- net EVDDA: now also R30.1, SV5.4; no longer R3.1, SV9.5
- net EVSS: now also SV5.1, SV9.7; no longer SV12.8, SV9.1
- net N$69: now also Q11.1; no longer Q11.2
- net N$70: now also Q11.2; no longer Q11.1
- net N$72: now also RQ.2; no longer R14.2
- net N$78: now also RQ.1; no longer R14.1
Other:
- moved on the sheet: C14, C15, C2, C24, C25, C3, C35, Q11

Commit message: Early drop for STM32PiBoard
Parts:
- L1, L2, L3, L4, L5, L6: device MyComponents:L-US0603 -> MyComponents:L-USL0603
Changed lines of the file:
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@@
 <setting verticaltext="up"/>
 </settings>
-<grid distance="0.05" unitdist="inch" unit="inch" style="lines" multiple="1" display="yes" altdistance="0.01" altunitdist="inch" altunit="inch"/>
+<grid distance="0.1" unitdist="inch" unit="inch" style="lines" multiple="1" display="no" altdistance="0.01" altunitdist="inch" altunit="inch"/>
 <layers>
 <layer number="1" name="Top" color="4" fill="1" visible="no" active="no"/>
@@
 <part name="SV19" library="MyComponents" deviceset="MA09-1" device="NO-PL"/>
 <part name="R10" library="MyComponents" deviceset="R-US" device="0805" value="10K"/>
-<part name="L1" library="MyComponents" deviceset="L-US" device="0603"/>
-<part name="L2" library="MyComponents" deviceset="L-US" device="0603"/>
-<part name="L3" library="MyComponents" deviceset="L-US" device="0603"/>
-<part name="L4" library="MyComponents" deviceset="L-US" device="0603"/>
-<part name="L5" library="MyComponents" deviceset="L-US" device="0603"/>
-<part name="L6" library="MyComponents" deviceset="L-US" device="0603"/>
+<part name="L1" library="MyComponents" deviceset="L-US" device="L0603"/>
+<part name="L2" library="MyComponents" deviceset="L-US" device="L0603"/>
+<part name="L3" library="MyComponents" deviceset="L-US" device="L0603"/>
+<part name="L4" library="MyComponents" deviceset="L-US" device="L0603"/>
+<part name="L5" library="MyComponents" deviceset="L-US" device="L0603"/>
+<part name="L6" library="MyComponents" deviceset="L-US" device="L0603"/>
 </parts>
 <sheets>

Commit message: Updated STM32 adapters
Parts:
- Q1, Q2, Q3: device MyComponents:Q-HC-46X -> MyComponents:Q-HSEHC-46X
- Q11, Q21: device MyComponents:Q-MC-306 -> MyComponents:Q-LSEMC-306
Changed lines of the file:
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@@
 <grid distance="0.1" unitdist="inch" unit="inch" style="lines" multiple="1" display="no" altdistance="0.01" altunitdist="inch" altunit="inch"/>
 <layers>
-<layer number="1" name="Top" color="4" fill="1" visible="no" active="no"/>
-<layer number="16" name="Bottom" color="1" fill="1" visible="no" active="no"/>
-<layer number="17" name="Pads" color="2" fill="1" visible="no" active="no"/>
-<layer number="18" name="Vias" color="2" fill="1" visible="no" active="no"/>
-<layer number="19" name="Unrouted" color="6" fill="1" visible="no" active="no"/>
-<layer number="20" name="Dimension" color="15" fill="1" visible="no" active="no"/>
-<layer number="21" name="tPlace" color="7" fill="1" visible="no" active="no"/>
-<layer number="22" name="bPlace" color="7" fill="1" visible="no" active="no"/>
-<layer number="23" name="tOrigins" color="15" fill="1" visible="no" active="no"/>
-<layer number="24" name="bOrigins" color="15" fill="1" visible="no" active="no"/>
-<layer number="25" name="tNames" color="7" fill="1" visible="no" active="no"/>
-<layer number="26" name="bNames" color="7" fill="1" visible="no" active="no"/>
-<layer number="27" name="tValues" color="7" fill="1" visible="no" active="no"/>
-<layer number="28" name="bValues" color="7" fill="1" visible="no" active="no"/>
+<layer number="1" name="Top" color="4" fill="1" visible="yes" active="no"/>
+<layer number="16" name="Bottom" color="1" fill="1" visible="yes" active="no"/>
+<layer number="17" name="Pads" color="2" fill="1" visible="yes" active="no"/>
+<layer number="18" name="Vias" color="2" fill="1" visible="yes" active="no"/>
+<layer number="19" name="Unrouted" color="6" fill="1" visible="yes" active="no"/>
+<layer number="20" name="Dimension" color="15" fill="1" visible="yes" active="no"/>
+<layer number="21" name="tPlace" color="7" fill="1" visible="yes" active="no"/>
+<layer number="22" name="bPlace" color="7" fill="1" visible="yes" active="no"/>
+<layer number="23" name="tOrigins" color="15" fill="1" visible="yes" active="no"/>
+<layer number="24" name="bOrigins" color="15" fill="1" visible="yes" active="no"/>
+<layer number="25" name="tNames" color="7" fill="1" visible="yes" active="no"/>
+<layer number="26" name="bNames" color="7" fill="1" visible="yes" active="no"/>
+<layer number="27" name="tValues" color="7" fill="1" visible="yes" active="no"/>
+<layer number="28" name="bValues" color="7" fill="1" visible="yes" active="no"/>
 <layer number="29" name="tStop" color="7" fill="3" visible="no" active="no"/>
 <layer number="30" name="bStop" color="7" fill="6" visible="no" active="no"/>
@@
 <layer number="35" name="tGlue" color="7" fill="4" visible="no" active="no"/>
 <layer number="36" name="bGlue" color="7" fill="5" visible="no" active="no"/>
-<layer number="37" name="tTest" color="7" fill="1" visible="no" active="no"/>
-<layer number="38" name="bTest" color="7" fill="1" visible="no" active="no"/>
+<layer number="37" name="tTest" color="7" fill="1" visible="yes" active="no"/>
+<layer number="38" name="bTest" color="7" fill="1" visible="yes" active="no"/>
 <layer number="39" name="tKeepout" color="4" fill="11" visible="no" active="no"/>
 <layer number="40" name="bKeepout" color="1" fill="11" visible="no" active="no"/>
@@
 <layer number="44" name="Drills" color="7" fill="1" visible="no" active="no"/>
 <layer number="45" name="Holes" color="7" fill="1" visible="no" active="no"/>
-<layer number="46" name="Milling" color="3" fill="1" visible="no" active="no"/>
-<layer number="47" name="Measures" color="7" fill="1" visible="no" active="no"/>
-<layer number="48" name="Document" color="7" fill="1" visible="no" active="no"/>
-<layer number="49" name="Reference" color="7" fill="1" visible="no" active="no"/>
-<layer number="50" name="dxf" color="7" fill="1" visible="no" active="no"/>
-<layer number="51" name="tDocu" color="7" fill="1" visible="no" active="no"/>
-<layer number="52" name="bDocu" color="7" fill="1" visible="no" active="no"/>
-<layer number="53" name="tGND_GNDA" color="7" fill="9" visible="no" active="no"/>
-<layer number="54" name="bGND_GNDA" color="1" fill="9" visible="no" active="no"/>
-<layer number="56" name="wert" color="7" fill="1" visible="no" active="no"/>
+<layer number="46" name="Milling" color="3" fill="1" visible="yes" active="no"/>
+<layer number="47" name="Measures" color="7" fill="1" visible="yes" active="no"/>
+<layer number="48" name="Document" color="7" fill="1" visible="yes" active="no"/>
+<layer number="49" name="Reference" color="7" fill="1" visible="yes" active="no"/>
+<layer number="50" name="dxf" color="7" fill="1" visible="yes" active="no"/>
+<layer number="51" name="tDocu" color="7" fill="1" visible="yes" active="no"/>
+<layer number="52" name="bDocu" color="7" fill="1" visible="yes" active="no"/>
+<layer number="53" name="tGND_GNDA" color="7" fill="9" visible="yes" active="no"/>
+<layer number="54" name="bGND_GNDA" color="1" fill="9" visible="yes" active="no"/>
+<layer number="56" name="wert" color="7" fill="1" visible="yes" active="no"/>
 <layer number="90" name="Modules" color="5" fill="1" visible="yes" active="yes"/>
 <layer number="91" name="Nets" color="2" fill="1" visible="yes" active="yes"/>
@@
 <part name="C30" library="MyComponents" deviceset="C-US" device="0805" value="0.1uF"/>
 <part name="C31" library="MyComponents" deviceset="C-US" device="0805" value="0.1uF"/>
-<part name="Q3" library="MyComponents" deviceset="Q-HC-46X" device="" value="HSE"/>
+<part name="Q3" library="MyComponents" deviceset="Q-HSE" device="HC-46X" value="HSE"/>
 <part name="C34" library="MyComponents" deviceset="C-US" device="0805" value="12pF"/>
 <part name="C33" library="MyComponents" deviceset="C-US" device="0805" value="12pF"/>
@@
 <part name="R21" library="MyComponents" deviceset="R-US" device="0805" value="10K"/>
 <part name="J2" library="MyComponents" deviceset="BUTTON-FSM14JRT" device=""/>
-<part name="Q2" library="MyComponents" deviceset="Q-HC-46X" device="" value="HSE"/>
+<part name="Q2" library="MyComponents" deviceset="Q-HSE" device="HC-46X" value="HSE"/>
 <part name="C24" library="MyComponents" deviceset="C-US" device="0805" value="12pF"/>
 <part name="C25" library="MyComponents" deviceset="C-US" device="0805" value="12pF"/>
 <part name="C22" library="MyComponents" deviceset="C-US" device="0805" value="4.7uF"/>
-<part name="Q21" library="MyComponents" deviceset="Q-MC-306" device="" value="LSE"/>
+<part name="Q21" library="MyComponents" deviceset="Q-LSE" device="MC-306" value="LSE"/>
 <part name="SV4" library="MyComponents" deviceset="MA05-2" device="" value="JTAG"/>
 <part name="C13" library="MyComponents" deviceset="C-US" device="0805" value="0.1uF"/>
@@
 <part name="R15" library="MyComponents" deviceset="R-US" device="0805" value="10K"/>
 <part name="J1" library="MyComponents" deviceset="BUTTON-FSM14JRT" device=""/>
-<part name="Q11" library="MyComponents" deviceset="Q-MC-306" device="" value="LSE"/>
-<part name="Q1" library="MyComponents" deviceset="Q-HC-46X" device="" value="HSE"/>
+<part name="Q11" library="MyComponents" deviceset="Q-LSE" device="MC-306" value="LSE"/>
+<part name="Q1" library="MyComponents" deviceset="Q-HSE" device="HC-46X" value="HSE"/>
 <part name="C2" library="MyComponents" deviceset="C-US" device="0805" value="12pF"/>
 <part name="C3" library="MyComponents" deviceset="C-US" device="0805" value="12pF"/>
