File: pcb/stm32_pi_board.brd (EAGLE design)
At the start: 84 x 56 mm, 102 parts, among them IC1 LMT86, IC10 REG1117, IC2 ESP-11, IC3 IS31AP2005, IC4 STM32F405RG, IC5 STF203-22, IC6 MIC5219-3.3, IC7 IS31AP2005, IC8 MIC5219-3.3, IC9 UDA1334ATS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

Commit message: PCB revision 1.3
Parts:
- added C40: 470 uF, MyComponents:CPOL2917
- moved L1 1.25 mm to (21.5, 44.2), flipped to the bottom, turned to 180 degrees
- moved L2 1.25 mm to (21.5, 46.8), flipped to the bottom, turned to 180 degrees
- moved C38 0.75 mm to (28.0, 38.0)
Connections:
- net GND: now also C40.-
- net VIN: now also C40.+
Routing:
- net GND: track 90.6 -> 92.8 mm, vias 21 -> 22
- net SD-D1: track 35.5 -> 36.9 mm
- net ESP-RX: track 29.7 -> 30.9 mm, vias 2 -> 1
- net ESP-TX: track 31.8 -> 32.9 mm, vias 2 -> 1
- net ESP-ON: track 49.5 -> 48.4 mm
- net SD-D0: track 33.8 -> 32.8 mm
- net VIN: track 52.5 -> 51.8 mm
- net ESP-RXI: track 14.5 -> 15.0 mm
Other:
- board text added: "STM32-Pi Board Revision 1.3 (C) Mikhail Kulesh"
- board text removed: "STM32-Pi Board Revision 1.2 (C) Mikhail Kulesh"

Commit message: Revision 1.3 of Stm32-Pi-Board
Parts:
- added OPH1: AMS3, photo-elements:VT900
- added R29: 4.7K, MyComponents:R0805
- C39: device rcl:C1206 -> MyComponents:C0805
- moved C16 6.04 mm to (17.0, 30.8), turned to 180 degrees
- moved SV1 1.00 mm to (12.0, 27.0), turned to 90 degrees
- turned RESET to 270 degrees
Connections:
- net GND: now also R29.1
- net PC0: now also OPH1.1, R29.2
- net VDD: now also OPH1.2
Routing:
- net SWDIO: track 50.5 -> 60.3 mm
- net VDD: track 127.1 -> 133.8 mm
- net NRST: track 49.0 -> 44.4 mm
- net PC0: track 26.5 -> 29.6 mm
- net SWCLK: track 50.0 -> 51.5 mm
Other:
- board text added: "CLK/ IO"
- board text added: "VCC"
- board text removed: "CL"
- board text removed: "IO"
- board text removed: "VCC/"

Commit message: Submitted PiBoard v1.3
Parts:
- moved D1 0.25 mm to (82.2, 43.5)
- moved R29 0.25 mm to (48.8, 49.2)
Connections:
- net GND: no longer D1.P$2
- net N$5: now also D1.P$1; no longer D1.P$3
- net N$75: now also D1.P$3; no longer D1.P$1
- net VDD: now also D1.P$2
Routing:
- net VDD: track 133.8 -> 162.5 mm
- net GND: track 92.8 -> 90.3 mm, vias 22 -> 21
